File: kicad/Sentinel 65.kicad_sch (KiCad schematic)
At the start: 0 parts

Commit message: More work in progress
Other:
- added sheet Audio Output (audio_output.kicad_sch)
- added sheet IO Connectors (io_connectors.kicad_sch)
- added sheet SD Slot (sd_slot.kicad_sch)
- added sheet Video Output (video_out.kicad_sch)
