File: kicad/vera.kicad_sch (KiCad schematic)
At the start: 0 parts

Commit message: More work in progress
Parts:
- added C10, C11, C14, C15, C16, C17, C19: 100nF, symbol Device:C
- added C12, C13, C18: 4.7uF, symbol Device:C
- added C21, C22: 10uF, Capacitor_SMD:C_0805_2012Metric, symbol Device:C_Small
- added C24, C25: 100nF, Capacitor_SMD:C_0603_1608Metric, symbol Device:C_Small
- added C3 (x2): 100nF, Capacitor_SMD:C_0402_1005Metric, symbol Device:C
- added JP1: Flash enable, Connector_PinHeader_2.54mm:PinHeader_1x02_P2.54mm_Vertical, symbol Jumper:Jumper_2_Open
- added L1: NRS4018T2R2MDGJ, Inductor_SMD:L_Bourns-SRN4018, symbol Device:L
- added R2: 1, Resistor_SMD:R_0603_1608Metric, symbol Device:R_Small
- added R3, R4, R5, R6: 47k, Resistor_SMD:R_0603_1608Metric, symbol Device:R_Small
- added U10: W25Q16JVSNIQ, Package_SO:SOIC-8_3.9x4.9mm_P1.27mm, symbol vera-module-rev4-rescue:W25Q32JVSS-Memory_Flash
- added U6: ICE40UP5K-SG48ITR, Package_DFN_QFN:QFN-48-1EP_7x7mm_P0.5mm_EP5.6x5.6mm, symbol FPGA_Lattice:ICE40UP5K-SG48ITR
- added U7: AP3417CKTR-G1, Package_TO_SOT_SMD:SOT-23-5, symbol vera-module:AP3417CKTR-G1
- added U8: 74CBTLV3126PW,118, Package_SO:TSSOP-14_4.4x5mm_P0.65mm, symbol vera-module:74CBTLV3126PW,118
- added U9: 74AHC00PW, Package_SO:TSSOP-14_4.4x5mm_P0.65mm, symbol 74xx:74HC00
- added X1: 25MHz, Oscillator:Oscillator_SMD_EuroQuartz_XO32-4Pin_3.2x2.5mm, symbol Oscillator:XO32
Connections:
- new net: U9.10, U9.13, U9.6
- new net: U9.3, U9.9
- new net: R5.2, U10.3 (IO2)
- new net: R6.2, U10.7 (IO3)
- new net: R3.2, R4.1, U7.5 (FB)
- new net: C21.1, R2.1, U7.1 (EN), U7.4 (VIN)
- new net: L1.1, U7.3 (LX)
- new net +1V2: C10.1, C11.1, C12.1, C13.1, C22.1, L1.2, R3.1, U6.29 (VCCPLL), U6.30 (VCC), U6.5 (VCC)
- new net +3.3V: C14.1, C15.1, C16.1, C17.1, C18.1, C19.1, C3.1, C3.1, U6.1 (VCCIO_2), U6.22 (SPI_VCCIO1), U6.24 (VPP_2V5), U6.33 (VCCIO_0), U8.14 (VCC), X1.1 (EN), X1.4 (V+)
- new net +3V3: C24.1, C25.1, R5.1, R6.1, U10.8 (VCC), U9.14 (VCC)
- new net +5V: R2.2
- new net A0: U6.40 (RGB1)
- new net A1: U6.39 (RGB0)
- new net A2: U6.37 (IOT_45a_G1)
- new net A3: U6.41 (RGB2)
- new net A4: U6.34 (IOT_44b)
- new net ADATA: U6.42 (IOT_51a)
- new net B0: U6.46 (IOB_0a)
- new net B1: U6.47 (IOB_2a)
- new net B2: U6.44 (IOB_3b_G6), U6.48 (IOB_4a)
- new net B3: U6.2 (IOB_6a)
- new net BCLK: U6.38 (IOT_50b)
- new net CDONE: JP1.2 (B), U6.7 (CDONE), U8.1 (1OE), U8.10 (3OE), U8.13 (4OE), U8.4 (2OE), U9.1, U9.12, U9.2
- new net D0: U6.27 (IOT_38b)
- new net D1: U6.26 (IOT_39a)
- new net D2: U6.25 (IOT_36b)
- new net D3: U6.23 (IOT_37a)
- new net D4: U6.21 (IOB_23b)
- new net D5: U6.20 (IOB_25b_G3)
- new net D6: U6.19 (IOB_29b)
- new net D7: U6.18 (IOB_31b)
- new net FPGA_MISO: U10.2 (DO(IO1)), U6.17 (IOB_33b_SPI_SI), U8.5 (2A)
- new net FPGA_MOSI: U10.5 (DI(IO0)), U6.14 (IOB_32a_SPI_SO), U8.2 (1A)
- new net FPGA_SCK: U10.6 (CLK), U6.15 (IOB_34a_SPI_SCK), U8.9 (3A)
- new net G0: U6.3 (IOB_9b)
- new net G1: U6.4 (IOB_8a)
- new net G2: U6.6 (IOB_13b)
- new net G3: U6.9 (IOB_16a)
- new net GND: C10.2, C11.2, C12.2, C13.2, C14.2, C15.2, C16.2, C17.2, C18.2, C19.2, C21.2, C22.2, C24.2, C25.2, C3.2, C3.2, JP1.1 (A), R4.2, U10.4 (GND), U6.49 (GND), U7.2 (GND), U8.7 (GND), U9.7 (GND), X1.2 (GND)
- new net LRCK: U6.43 (IOT_49a)
- new net MISO: U8.6 (2B)
- new net MOSI: U8.3 (1B)
- new net R0: U6.10 (IOB_18a)
- new net R1: U6.11 (IOB_20a)
- new net R2: U6.12 (IOB_22a)
- new net R3: U6.13 (IOB_24a)
- new net SCK: U8.8 (3B)
- new net SYSCLK: U6.35 (IOT_46b_G0), X1.3 (OUT)
- new net VSYNC: U6.45 (IOB_5b)
- new net ~{FLASH_SS}: U10.1 (~{CS}), U9.8
- new net ~{FPGA_SS}: U6.16 (IOB_35b_SPI_SS), U9.4, U9.5
- new net ~{IRQ}: U6.32 (IOT_43a)
- new net ~{RD}: U6.36 (IOT_48b)
- new net ~{RES}: U6.8 (~{CRESET})
- new net ~{SD_SS}: U8.12 (4A), U9.11
- new net ~{SS}: U8.11 (4B)
- new net ~{VERA}: U6.28 (IOT_41a)
- new net ~{WR}: U6.31 (IOT_42b)
