File: kicad/Sentinel 65 V2/Sentinel 65 V2.kicad_sch (KiCad schematic)
At the start: 169 parts, among them J1 SNES Controller, J10 Conn_01x02, J12 LEFT, J13 RIGHT, J14 USB_C_Receptacle_PowerOnly_6P, J15 Conn_01x02, J2 SNES Controller, J3 Conn_02x12_Odd_Even, J4 2x32 2.54mm Card Edge Connect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, J5 Internal Control Header (Opti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, J6 Conn_02x11_Odd_Even, J7 SD_Card, J8 FPGA_PROG, J9 SVGA Connector, SW1 SW_Push, SW3 SW_Push, U1 ATF22LV10C, U10 TLV9062xD, U11 LM1086IT-3.3, U12 MCP1316MT-33LE/OT, U2 SST39LF040-55-4C-NHE-T, U3 W65C265S8PLG-8, U4 IS61WV5128EDBLL-10TLI, U5 W25Q16JVSNIQ, U6 74CBTLV3126PW,118, U7 AP7361C-12E, U8 ICE40UP5K-SG48ITR, U9 WM8524CGEDT, X1 32.768KHz, X2 8Mhz, X3 25MHz

Commit message: Added programmable clock generator
Parts:
- removed C24, C25: 100nF, Capacitor_SMD:C_0402_1005Metric, symbol Device:C
- removed X1: 32.768KHz, Oscillator:Oscillator_SMD_EuroQuartz_XO91-4Pin_7.0x5.0mm, symbol Oscillator:XO91
- removed X2: 8Mhz, Oscillator:Oscillator_SMD_EuroQuartz_XO91-4Pin_7.0x5.0mm, symbol Oscillator:XO91
- removed X3: 25MHz, Oscillator:Oscillator_SMD_EuroQuartz_XO91-4Pin_7.0x5.0mm, symbol Oscillator:XO91
- added R10, R9: 3.3kΩ, Resistor_SMD:R_0402_1005Metric, symbol Device:R
- added U8: Si5351A, Package_SO:MSOP-10-1EP_3x3mm_P0.5mm_EP1.68x1.88mm, symbol Oscillator:Si5351A
- added Y1: 25MHz, symbol Device:Crystal
- renumbered C27 to C24, C28 to C25, C29 to C26, C30 to C27, C31 to C28, C32 to C29, C33 to C30, C34 to C31, C35 to C32, C36 to C33, C37 to C34, C38 to C35, C39 to C36, C40 to C37, C41 to C38, C42 to C39, C43 to C40, D4 to D1, D12 to D10, D13 to D11, D5 to D2, D2 to D3, D3 to D4, D6 to D5, D8 to D6, D9 to D7, D7 to D8, D10 to D9, J15 to J10, J10 to J11, R9 to R11, R10 to R12, R11 to R13, R12 to R14, R13 to R15, R14 to R16, R15 to R17, R16 to R18, R17 to R19, R18 to R20, R19 to R21, R20 to R22, R21 to R23, R22 to R24, R23 to R25, R24 to R26, R25 to R27, R26 to R28, R27 to R29, R28 to R30, R29 to R31, R30 to R32, R31 to R33, R32 to R34, R33 to R35, R34 to R36, R35 to R37, R36 to R38, R38 to R39, R39 to R40, R40 to R41, R41 to R42, R42 to R43, R43 to R44, R44 to R45, R51 to R46, R52 to R47, R45 to R48, R46 to R49, R47 to R50, R48 to R51, R49 to R52, R50 to R53, R53 to R54, R54 to R55, R63 to R56, R64 to R57, R55 to R58, R56 to R59, R57 to R60, R58 to R61, R59 to R62, R60 to R63, R61 to R64, R62 to R65, R65 to R66, R66 to R67, R67 to R68, R70 to R69, R68 to R70, R69 to R71, R71 to R72, R72 to R73, R73 to R74, R74 to R75, R75 to R76, R76 to R77, R77 to R78, R78 to R79, R79 to R80, SW3 to SW2, U9 to U10, U10 to U11, U11 to U12, U12 to U13, U8 to U9
Connections:
- net +3.3V: now also R10.1, R9.1, U8.1 (VCC), U8.7 (VCCO)
- net CLK: now also U8.10 (GND)
- net FCLK: now also U8.9 (CLK1)
- net GND: now also U8.10 (GND)
- net I2C_SCL: now also R9.2, U8.4 (SCL)
- net I2C_SDA: now also R10.2, U8.2 (XA)
- net SYSCLK: now also U8.6 (CLK2)
- new net: U8.2 (XA), Y1.1
- new net: U8.3 (XB), Y1.2
Other:
- note removed: "CPU Osclillators must have a 5nS or lower rise/fall time"

Commit message: Switched glue logic to ATF1502 TQFP-44, added JTAG header
Parts:
- removed C5: 100nF, Capacitor_SMD:C_0402_1005Metric, symbol Device:C
- removed J3: Conn_02x12_Odd_Even, symbol Connector_Generic:Conn_02x12_Odd_Even
- removed J8: FPGA_PROG, Connector_PinHeader_2.54mm:PinHeader_1x08_P2.54mm_Vertical, symbol Connector_Generic:Conn_01x08
- removed R21: 10kΩ, Resistor_SMD:R_0402_1005Metric, symbol Device:R
- removed U1: ATF22LV10C, Package_DIP:DIP-24_W8.89mm_SMDSocket_LongPads, symbol Logic_Programmable:ATF22LV10C
- added C1: 100nF, Capacitor_SMD:C_0402_1005Metric, symbol Device:C
- added J10: Conn_02x04_Odd_Even, symbol Connector_Generic:Conn_02x04_Odd_Even
- added J3: Conn_02x14_Odd_Even, symbol Connector_Generic:Conn_02x14_Odd_Even
- added J4: JTAG Header, symbol Connector_Generic:Conn_02x05_Odd_Even
- added R1: 10kΩ, Resistor_SMD:R_0402_1005Metric, symbol Device:R
- added U4: ATF1502ASV-xAx44, Package_QFP:TQFP-44_10x10mm_P0.8mm, symbol CPLD_Microchip:ATF1502ASV-xAx44
- renumbered C1 to C2, C2 to C3, C3 to C4, C4 to C5, D3 to D1, D4 to D2, D1 to D3, D2 to D4, D8 to D6, D9 to D7, D6 to D8, D7 to D9, J10 to J11, J11 to J12, J12 to J13, J13 to J14, J14 to J15, J4 to J5, J5 to J6, J6 to J7, J7 to J8, R9 to R10, R10 to R11, R11 to R12, R12 to R13, R13 to R14, R14 to R15, R15 to R16, R16 to R17, R17 to R18, R18 to R19, R1 to R2, R19 to R20, R20 to R21, R2 to R3, R3 to R4, R48 to R46, R49 to R47, R50 to R48, R51 to R49, R4 to R5, R52 to R50, R53 to R51, R46 to R52, R47 to R53, R58 to R56, R59 to R57, R60 to R58, R61 to R59, R5 to R6, R62 to R60, R63 to R61, R64 to R62, R65 to R63, R66 to R64, R67 to R65, R56 to R66, R57 to R67, R6 to R7, R7 to R8, R8 to R9, U2 to U1, U3 to U2, U4 to U3
Connections:
- net +3.3V: now also C1.1, J3.2 (Pin_2), J4.4 (Pin_4), R1.1, U4.17 (VCC), U4.29 (VCC), U4.41 (VCC), U4.9 (VCC)
- net A0: now also J3.20 (Pin_20)
- net A1: now also J3.19 (Pin_19)
- net A19: now also U4.27 (I/O)
- net A2: now also J3.18 (Pin_18)
- net A20: now also U4.28 (I/O)
- net A21: now also U4.30 (I/O)
- net A3: now also J3.17 (Pin_17)
- net A5: now also U4.25 (I/O)
- net BL0: now also J10.1 (Pin_1)
- net BL1: now also J10.3 (Pin_3)
- net BL2: now also J10.5 (Pin_5)
- net BL3: now also J10.7 (Pin_7)
- net CDONE: now also U4.38 (I/OE1/Vpp)
- net D0: now also J3.28 (Pin_28)
- net D1: now also J3.27 (Pin_27)
- net D2: now also J3.26 (Pin_26)
- net D3: now also J3.25 (Pin_25)
- net D4: now also J3.24 (Pin_24)
- net D5: now also J3.23 (Pin_23)
- net D6: now also J3.22 (Pin_22)
- net D7: now also J3.21 (Pin_21)
- net FPGA_MISO: now also J3.6 (Pin_6)
- net FPGA_MOSI: now also J3.4 (Pin_4)
- net FPGA_SCK: now also J3.5 (Pin_5)
- net GND: now also C1.2, J10.2 (Pin_2), J10.4 (Pin_4), J10.6 (Pin_6), J10.8 (Pin_8), J3.1 (Pin_1), J4.10 (Pin_10), J4.2 (Pin_2), U4.16 (GND), U4.24 (GND), U4.36 (GND), U4.4 (GND)
- net I2C_SCL: now also J3.8 (Pin_8)
- net I2C_SDA: now also J3.10 (Pin_10)
- net IRQ3: now also U4.5 (I/O/PD1)
- net PHI2: now also J3.13 (Pin_13), U4.37 (I/GCLK1)
- net RXD: now also J3.9 (Pin_9)
- net R/~{W}: now also U4.42 (I/O)
- net TXD: now also J3.7 (Pin_7)
- net ~{CLOCK}: now also J3.14 (Pin_14), U4.12 (I/O)
- net ~{FLASH_SS}: now also R1.2, U4.3 (I/O)
- net ~{FPGA_SS}: now also J3.3 (Pin_3), U4.40 (I/OE2/GCLK2)
- net ~{HIROM}: now also U4.33 (I/O)
- net ~{IO}1: now also U4.34 (I/O)
- net ~{IRQ}2: now also J3.12 (Pin_12)
- net ~{IRQ}3: now also U4.35 (I/O/GCLK3)
- net ~{LOROM}: now also U4.31 (I/O)
- net ~{RD}: now also J3.15 (Pin_15), U4.10 (I/O)
- net ~{RES}: now also J3.11 (Pin_11), U4.39 (I/GCLR)
- net ~{ROM}0: now also U4.13 (I/O)
- net ~{ROM}1: now also U4.14 (I/O)
- net ~{SD_SS}: now also U4.2 (I/O)
- net ~{VERA}: now also U4.11 (I/O)
- net ~{WR}: now also J3.16 (Pin_16), U4.8 (I/O)
- new net TCK: J4.1 (Pin_1), U4.26 (I/O/TCK)
- new net TDI: J4.9 (Pin_9), U4.1 (I/O/TDI)
- new net TDO: J4.3 (Pin_3), U4.32 (I/O/TDO)
- new net TMS: J4.5 (Pin_5), U4.7 (I/O/TMS)
- no-connect marks 14 -> 26
Other:
- note added: "Clock Defaults: CLK: 32.768KHz TOD clock FCLK: 8MHz+ fast clock SYSCLK: 25MHz VERA clock"
- note added: "Clock Generator"
- note added: "Supplemental Glue Logic"
- note removed: "ATF22LV10C-10JU Glue Logic"
- note removed: "Future DV board options may need to use the pixel clock from the VERA directly; to prepare for that eventuality, a solderable jumper is provided which can be used to disconnect PHI2 from the VERA, and connect that pin to the DV header."
- note removed: "This revision of the design uses a PLCC-84 CPU and a DIP GAL, because they are what I have in stock at the moment. The next revision will switch those to equivalent parts in SMD packages: QFP-100 for the CPU, PLCC for the ATF22LV10C."
- note removed: "VERA Clock"
- moved on the sheet: C2, C23, C3, C4, C5, D3, D4, D8, D9, JP1, R10, R11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

Commit message: Removed DV header, deferred to Rev1. Updated PDF schematic.
Parts:
- removed J7: Conn_02x11_Odd_Even, symbol Connector_Generic:Conn_02x11_Odd_Even
- removed JP1: SolderJumper_3_Bridged12, Jumper:SolderJumper-3_P1.3mm_Bridged12_RoundedPad1.0x1.5mm, symbol Jumper:SolderJumper_3_Bridged12
Connections:
- net VCLK is gone; now on net PHI2: U9.36 (IOT_48b)
- net ~{FLASH_SS}: now also J3.3 (Pin_3)
- net ~{FPGA_SS}: no longer J3.3 (Pin_3)
Other:
- note added: "The CPU is a PLCC-84 in an SMD socket"
- note removed: "DV Header (Optional)"
- moved on the sheet: R23, R24, R29, R30, R35, R36, R37, R38, R39, R40, R41, R42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

Commit message: Added project-specific library
Parts:
- C1, C10, C11, C12, C13, C14, C15, C16, C17, C18, C19, C2, C20, C21, C22, C23, C26, C28, C3, C32, C33, C34, C35, C36, C37, C4, C40, C5, C6, C7, C8, C9: symbol Device:C -> Sentinel 65X:C
- C24, C25, C27, C29, C30, C31, C38, C39: symbol Device:C_Polarized -> Sentinel 65X:C_Polarized
- D1, D10, D11, D2, D5, D6, D7: symbol Diode:PESD3V3L1BA-N -> Sentinel 65X:PESD3V3L1BA-N
- D3, D4, D8, D9: symbol Device:LED -> Sentinel 65X:LED
- H1, H2, H3, H4, H5, H6: symbol Mechanical:MountingHole_Pad -> Sentinel 65X:MountingHole_Pad
- J1, J2: symbol Connector_Generic:Conn_01x07 -> Sentinel 65X:Conn_01x07
- J10: symbol Connector_Generic:Conn_02x04_Odd_Even -> Sentinel 65X:Conn_02x04_Odd_Even
- J11, J12: symbol Connector_Generic:Conn_01x02 -> Sentinel 65X:Conn_01x02
- J13, J14: symbol Connector:Conn_Coaxial -> Sentinel 65X:Conn_Coaxial
- J15: symbol Connector:USB_C_Receptacle_PowerOnly_6P -> Sentinel 65X:USB_C_Receptacle_PowerOnly_6P
- J3: symbol Connector_Generic:Conn_02x14_Odd_Even -> Sentinel 65X:Conn_02x14_Odd_Even
- J4, J6: symbol Connector_Generic:Conn_02x05_Odd_Even -> Sentinel 65X:Conn_02x05_Odd_Even
- J5: symbol Connector_Generic:Conn_02x32_Row_Letter_First -> Sentinel 65X:Conn_02x32_Row_Letter_First
- J8: symbol Connector:SD_Card -> Sentinel 65X:SD_Card
- J9: symbol Connector:DE15_Receptacle_HighDensity_MountingHoles -> Sentinel 65X:DE15_Receptacle_HighDensity_MountingHoles
- R1, R10, R11, R12, R13, R14, R15, R16, R17, R18, R19, R2, R20, R21, R22, R23, R24, R25, R26, R27, R28, R29, R3, R30, R31, R32, R33, R34, R35, R36, R37, R38, R39, R4, R40, R41, R42, R43, R44, R45, R46, R47, R48, R49, R5, R50, R51, R52, R53, R54, R55, R56, R57, R58, R59, R6, R60, R61, R62, R63, R64, R65, R66, R67, R68, R69, R7, R70, R71, R72, R73, R74, R75, R76, R77, R78, R79, R8, R80, R9: symbol Device:R -> Sentinel 65X:R
- SW1, SW2: symbol Switch:SW_Push -> Sentinel 65X:SW_Push
- U1: symbol Memory_Flash:SST39LF040-55-4C-NHE-T -> Sentinel 65X:SST39LF040-55-4C-NHE-T
- U10: symbol Analog_DAC:WM8524CGEDT -> Sentinel 65X:WM8524CGEDT
- U11: symbol Amplifier_Operational:TLV9062xD -> Sentinel 65X:TLV9062xD_1
- U11: symbol Amplifier_Operational:TLV9062xD -> Sentinel 65X:TLV9062xD
- U11: symbol Amplifier_Operational:TLV9062xD -> Sentinel 65X:TLV9062xD_2
- U12: symbol Regulator_Linear:LM1086IT-3.3 -> Sentinel 65X:LM1086IT-3.3
- U13: symbol Power_Supervisor:MCP1316MT-33LE/OT -> Sentinel 65X:MCP1316MT-33LE/OT
- U2: symbol Western Design Center:W65C265S8PLG-8 -> Sentinel 65X:W65C265S8PLG-8
- U3: symbol Memory_RAM:IS61WV5128EDBLL-10TLI -> Sentinel 65X:IS61WV5128EDBLL-10TLI
- U4: symbol CPLD_Microchip:ATF1502ASV-xAx44 -> Sentinel 65X:ATF1502ASV-xAx44
- U5: symbol Memory_Flash:W25Q16JVSNIQ -> Sentinel 65X:W25Q16JVSNIQ
- U6: symbol 74xx:74CBTLV3126PW,118 -> Sentinel 65X:74CBTLV3126PW,118
- U7: symbol Regulator_Linear:AP7361C-12E -> Sentinel 65X:AP7361C-12E
- U8: symbol Oscillator:Si5351A -> Sentinel 65X:Si5351A
- U9: symbol FPGA_Lattice:ICE40UP5K-SG48ITR -> Sentinel 65X:ICE40UP5K-SG48ITR
- Y1: symbol Device:Crystal -> Sentinel 65X:Crystal

Commit message: Added FPGA CDONE and reset pins to CPU GPIO. Added CDONE indicator LED.
Parts:
- removed D3: LED0, symbol Sentinel 65X:LED
- removed D4: LED2, symbol Sentinel 65X:LED
- removed D8: LED1, symbol Sentinel 65X:LED
- removed D9: LED3, symbol Sentinel 65X:LED
- removed J10: Conn_02x04_Odd_Even, symbol Sentinel 65X:Conn_02x04_Odd_Even
- removed R44, R60, R61, R62, R63: 47kΩ, Resistor_SMD:R_0402_1005Metric, symbol Sentinel 65X:R
- removed R52, R53, R66, R67: 1kΩ, Resistor_SMD:R_0402_1005Metric, symbol Sentinel 65X:R
- added D3, D4, D8: LED, symbol Device:LED
- added J7: Conn_02x03_Odd_Even, symbol Connector_Generic:Conn_02x03_Odd_Even
- added R81: 3.3kΩ, Resistor_SMD:R_0402_1005Metric, symbol Sentinel 65X:R
- R41, R42, R43: value 47kΩ -> 1kΩ
Connections:
- net BL3 is gone; now on net FPGA_MISO: U2.75 (P45)
- net +3.3V: no longer R41.1, R42.1, R43.1
- net BL0: now also R43.2, U2.77 (P47); no longer R41.2, U2.72 (P42)
- net BL1: now also U2.76 (P46); no longer U2.73 (P43)
- net CDONE: now also R41.2, U2.73 (P43)
- net FPGA_MISO: no longer U2.11 (P67)
- net FPGA_MOSI: now also U2.74 (P44); no longer U2.9 (P65)
- net GND: now also D3.1 (K), D4.1 (K), D8.1 (K), J7.2 (Pin_2), J7.4 (Pin_4), J7.6 (Pin_6)
- net I2C_SCL: now also U2.11 (P67); no longer U2.77 (P47)
- net I2C_SDA: now also U2.9 (P65); no longer U2.76 (P46)
- net ~{RES}: no longer U9.8 (~{CRESET})
- removed net BL2: R43.2, U2.74 (P44)
- new net: D8.2 (A), J7.1 (Pin_1), R43.1
- new net: D4.2 (A), J7.3 (Pin_3), R42.1
- new net: D3.2 (A), J7.5 (Pin_5), R41.1
- new net ~{FPGA_RES}: R81.2, U2.72 (P42), U9.8 (~{CRESET})
Other:
- note added: "Status Lights"
- note removed: "Blinkenlights"
- note removed: "Hardware Revision Code"
- note removed: "When set to inputs (the default state), BL[0..3] are connected to weak pullup or pulldown resistors, to encode the hardware revision for software to detect. When set to outputs, they control the "blinkenlight" LEDs. HHHH: Rev0 HHHL: Rev1 HHLH: Rev2 HHLL: Rev3 (etc.)"
- moved on the sheet: R70, R71
