File: kicad/Sentinel 65X - Prototype 4/Sentinel 65X - Prototype 4.kicad_sch (KiCad schematic)
At the start: 126 parts, among them J1 SVGA Connector, J10 Barrel_Jack_MountingPin, J11 Controller 1, J12 Controller 1, J2 2x32 2.54mm Card Edge Connect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, J3 2x32 2.54mm Card Edge Connect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, J4 Conn_02x08_Odd_Even, J5 Conn_01x02, J6 Conn_01x02, J7 Conn_01x02, J8 Conn_02x14_Odd_Even, J9 DM1AA-SF-PEJ(82), SW1 SW_Push, SW2 SW_Push, SW3 SW_Push, U1 Upduino_VERA, U2 W65C265S8PLG-8, U3 AS6C4008-55PCN, U4 SST39LF040-55-4C-NHE-T, U5 GY-PCM5102, U6 ATF22LV10C-10JU, U7 L7805CV-DG, U8 LM1085IT-3.3/NOPB, X1 ECS-327MVATX-5-CN-TR, X2 KC5032K8.00000C1GE00, X3 ECS-3963-250-BN-TR

Commit message: Updated schematics and PCB files for prototype 4
Parts:
- removed C18, C19: 10µF, Capacitor_THT:CP_Radial_D5.0mm_P2.50mm, symbol Device:C_Polarized
- removed D6: 1.5KE15CA, Diode_THT:D_DO-201AE_P15.24mm_Horizontal, symbol Diode:1.5KExxCA
- removed D7: VS-KBPC601, Diode_THT:Diode_Bridge_Vishay_KBPC6, symbol Device:D_Bridge_+A-A
- removed F1: 0ZRG0120FF1E, Fuse:Fuse_BelFuse_0ZRE0005FF_L8.3mm_W3.8mm, symbol Device:Fuse
- removed H2: MountingHole_Pad, MountingHole:MountingHole_3.2mm_M3_DIN965_Pad, symbol Mechanical:MountingHole_Pad
- removed J10: Barrel_Jack_MountingPin, Connector_BarrelJack:BarrelJack_Horizontal, symbol Connector:Barrel_Jack_MountingPin
- removed U7: L7805CV-DG, Package_TO_SOT_THT:TO-220-3_Vertical, symbol Regulator_Linear:L7805
- removed U8: LM1085IT-3.3/NOPB, Package_TO_SOT_THT:TO-220-3_Vertical, symbol Regulator_Linear:LM1085-3.3
- added C18, C19, C20, C23: 100nF, Capacitor_SMD:C_0805_2012Metric, symbol Device:C
- added C21, C22: 47pF, Capacitor_SMD:C_0805_2012Metric, symbol Device:C
- added J10: USB_C_Receptacle_USB2.0_14P, Connector_USB:USB_C_Receptacle_GCT_USB4085, symbol Connector:USB_C_Receptacle_USB2.0_14P
- added R65, R66: 10KΩ, Resistor_SMD:R_0805_2012Metric, symbol Device:R
- added R67, R68: 5.1KΩ, Resistor_SMD:R_0805_2012Metric, symbol Device:R
- added R69, R70: 270Ω, Resistor_SMD:R_0805_2012Metric, symbol Device:R
- added U7: NCP1117-3.3_SOT223, Package_TO_SOT_SMD:SOT-223-3_TabPin2, symbol Regulator_Linear:NCP1117-3.3_SOT223
- added U8: FT230XS, Package_SO:SSOP-16_3.9x4.9mm_P0.635mm, symbol Interface_USB:FT230XS
- added X4: ECS-5032MV-40-CN-TR, Oscillator:Oscillator_SMD_EuroQuartz_XO53-4Pin_5.0x3.2mm_HandSoldering, symbol Oscillator:XO53
- C16, C17: footprint Capacitor_THT:CP_Radial_D5.0mm_P2.50mm -> Capacitor_SMD:CP_Elec_4x5.4; now in the parts list
Connections:
- net +3.3V: now also C17.1, C19.1, C20.1, C23.1, R65.2, U7.2 (VO), U8.10 (3V3OUT), U8.11 (~{RESET}), U8.12 (VCC), U8.3 (VCCIO), X4.4 (V+); no longer X2.1 (EN)
- net +5V: now also C16.1, C18.1, J10.A4 (VBUS), J10.A9 (VBUS), J10.B4 (VBUS), J10.B9 (VBUS), U7.3 (VI); no longer C17.1
- net CTS: now also R70.2
- net FCLK: now also X4.3 (OUT)
- net GND: now also C18.2, C19.2, C20.2, C21.2, C22.2, C23.2, J10.A1 (GND), J10.A12 (GND), J10.B1 (GND), J10.B12 (GND), J10.S1 (SHIELD), R66.2, R67.2, R68.2, U7.1 (GND), U8.13 (GND), U8.5 (GND), X4.2 (GND)
- net RTS: now also U8.6 (~{CTS})
- net RXD: now also R69.2
- net TXD: now also U8.4 (RXD)
- net FCLK_SLOW: now reaches U2.6 (P62)
- net FCLK_SLOW: now also R65.1, X4.1 (EN)
- net FCLK_FAST: now reaches U2.9 (P65)
- net FCLK_FAST: now also X2.1 (EN), R66.1
- new net: J10.A5 (CC1), R67.1
- new net: J10.B5 (CC2), R68.1
- new net: R69.1, U8.1 (TXD)
- new net: R70.1, U8.2 (~{RTS})
- new net D+: C21.1, J10.A6 (D+), J10.B6 (D+), U8.8 (USBDP)
- new net D-: C22.1, J10.A7 (D-), J10.B7 (D-), U8.9 (USBDM)
- no-connect marks 35 -> 36
Other:
- note removed: "Power Supply"
- moved on the sheet: C11, C12, C13, X1, X3
