File: kicad/Sentinel 65X - Prototype 4 V2/Glue Logic.kicad_sch (KiCad schematic)
At the start: 30 parts, among them J1 AVR ICSP, SW1 6x6mm tact, U7 ATF22LV10C-10JU, U8 Si5351A-B-GT, U9 ATmega88P-20A, X1 ECS-250-6-37B2-AGY-TR

Commit message: Updated prototype 4V2 schematic
Parts:
- added R50: 3.3KΩ, Resistor_SMD:R_0402_1005Metric, symbol Device:R
Connections:
- net +3.3V: now also R50.1
- net ~{CART}: now reaches U9.14 (PB2)
- net ~{CART}: now also R50.2
- no-connect marks 8 -> 7
Other:
- moved on the sheet: R20, R21, R22, R23, R24, R25, R26, R27, R28, R29
